Commit message: 所有宇树接口都改成ros2话题接口，原先宇树仿真输出信息也桥接到ros2话题接口

File: src/descriptions/unitree/go2_description/xacro/ros2_control.xacro (robot description, xacro)
@@ -4,7 +4,12 @@
 		<hardware>
 			<plugin>hardware_unitree_mujoco/HardwareUnitree</plugin>
-<!--			<param name="domain">0</param>-->
-<!--			<param name="network_interface">enp46s0</param>-->
-<!--			<param name="show_foot_force">true</param>-->
+			<!-- All IO via ROS topics (DDS-free) -->
+			<param name="state_joint_topic">/joint_states</param>
+			<param name="state_imu_topic">/imu</param>
+			<param name="state_foot_force_topic">/foot_force</param>
+			<param name="state_odometry_topic">/odometry</param>
+			<param name="command_joint_topic">/joint_command</param>
+			<param name="command_kp_topic">/joint_kp</param>
+			<param name="command_kd_topic">/joint_kd</param>
 		</hardware>
 		<joint name="FR_hip_joint">

File: src/descriptions/unitree/mybot_description/urdf/robot.urdf (robot description, URDF)
Before this commit: robot mybot, 21 links, 20 joints
Links:
- removed link body
- added link trunk, mass 5.3036; collision box size=0.3762 0.0935 0.114; visual mesh filename=package://mybot_description/meshes/body.STL
- link FL_calf: geometry collision box size=0.213 0.016 0.016; visual mesh filename=package://mybot_description/meshes/FL_calf.STL
- link FL_foot: geometry collision sphere radius=0.02; visual mesh filename=package://mybot_description/meshes/FL_foot.STL
- link FL_hip: geometry collision cylinder length=0.04 radius=0.046; visual mesh filename=package://mybot_description/meshes/FL_hip.STL
- link FL_thigh: geometry collision box size=0.213 0.0245 0.034; visual mesh filename=package://mybot_description/meshes/FL_thigh.STL
- link FR_calf: geometry collision box size=0.213 0.016 0.016; visual mesh filename=package://mybot_description/meshes/FR_calf.STL
- link FR_foot: geometry collision sphere radius=0.02; visual mesh filename=package://mybot_description/meshes/FR_foot.STL
- link FR_hip: mass 0.645332324862741 -> 0.62455; geometry collision cylinder length=0.04 radius=0.046; visual mesh filename=package://mybot_description/meshes/FR_hip.STL
- link FR_thigh: mass 1.10704185501149 -> 1.107; geometry collision box size=0.213 0.0245 0.034; visual mesh filename=package://mybot_description/meshes/FR_thigh.STL
- link RL_calf: geometry collision box size=0.213 0.016 0.016; visual mesh filename=package://mybot_description/meshes/RL_calf.STL
- link RL_foot: geometry collision sphere radius=0.02; visual mesh filename=package://mybot_description/meshes/RL_foot.STL
- link RL_hip: mass 0.603770938189494 -> 0.62455; geometry collision cylinder length=0.04 radius=0.046; visual mesh filename=package://mybot_description/meshes/RL_hip.STL
- link RL_thigh: mass 1.10704185443719 -> 1.107; geometry collision box size=0.213 0.0245 0.034; visual mesh filename=package://mybot_description/meshes/RL_thigh.STL
- link RR_calf: mass 0.292483071997453 -> 0.292483071997452; geometry collision box size=0.213 0.016 0.016; visual mesh filename=package://mybot_description/meshes/RR_calf.STL
- link RR_foot: geometry collision sphere radius=0.02; visual mesh filename=package://mybot_description/meshes/RR_foot.STL
- link RR_hip: mass 0 -> 0.62455; geometry collision cylinder length=0.04 radius=0.046; visual mesh filename=package://mybot_description/meshes/RR_hip.STL
- link RR_thigh: mass 1.10704185429829 -> 1.107; geometry collision box size=0.213 0.0245 0.034; visual mesh filename=package://mybot_description/meshes/RR_thigh.STL
Joints:
- joint FL_calf_joint: limit lower=-2.7 upper=-0.6 effort=33.5 velocity=21 -> lower=-2.7227 upper=-0.83776 effort=35.55 velocity=20.06
- joint FL_foot_fixed: origin xyz=0.0015191 -0.00024999 -0.22467 rpy=0 0 0 -> xyz=0.0015191 -0.00025 -0.22467 rpy=0 0 0
- joint FL_hip_joint: limit lower=-0.48 upper=0.48 effort=33.5 velocity=21 -> lower=-1.0472 upper=1.0472 effort=23.7 velocity=30.1; parent body -> trunk
- joint FL_thigh_joint: limit lower=-1.44 upper=1.44 effort=33.5 velocity=21 -> lower=-1.5708 upper=3.4907 effort=23.7 velocity=30.1
- joint FR_calf_joint: limit lower=-2.7 upper=-0.6 effort=33.5 velocity=21 -> lower=-2.7227 upper=-0.83776 effort=35.55 velocity=20.06
- joint FR_foot_fixed: origin xyz=0.0015191 0.00025002 -0.22467 rpy=0 0 0 -> xyz=0.0015191 0.00025 -0.22467 rpy=0 0 0
- joint FR_hip_joint: limit lower=-0.48 upper=0.48 effort=33.5 velocity=21 -> lower=-1.0472 upper=1.0472 effort=23.7 velocity=30.1; parent body -> trunk
- joint FR_thigh_joint: limit lower=-1.44 upper=1.44 effort=33.5 velocity=21 -> lower=-1.5708 upper=3.4907 effort=23.7 velocity=30.1
- joint RL_calf_joint: limit lower=-2.7 upper=-0.6 effort=33.5 velocity=21 -> lower=-2.7227 upper=-0.83776 effort=35.55 velocity=20.06
- joint RL_foot_fixed: origin xyz=0.0015191 -0.00024998 -0.22467 rpy=0 0 0 -> xyz=0.0015191 -0.00025 -0.22467 rpy=0 0 0
- joint RL_hip_joint: limit lower=-0.48 upper=0.48 effort=33.5 velocity=21 -> lower=-1.0472 upper=1.0472 effort=23.7 velocity=30.1; origin xyz=-0.2146 0.062 -0.071 rpy=0 0 0 -> xyz=-0.0946 0.062 -0.071 rpy=0 0 0; parent body -> trunk
- joint RL_thigh_joint: limit lower=-1.48 upper=1.48 effort=33.5 velocity=21 -> lower=-1.5708 upper=3.4907 effort=23.7 velocity=30.1
- joint RR_calf_joint: limit lower=-2.7 upper=-0.6 effort=33.5 velocity=21 -> lower=-2.7227 upper=-0.83776 effort=35.55 velocity=20.06
- joint RR_foot_fixed: origin xyz=0.0015191 0.00025002 -0.22467 rpy=0 0 0 -> xyz=0.0015191 0.00025 -0.22467 rpy=0 0 0
- joint RR_hip_joint: limit lower=-0.48 upper=0.48 effort=33.5 velocity=21 -> lower=-1.0472 upper=1.0472 effort=23.7 velocity=30.1; origin xyz=-0.2146 -0.062 -0.071 rpy=0 0 0 -> xyz=-0.0946 -0.062 -0.071 rpy=0 0 0; parent body -> trunk
- joint RR_thigh_joint: limit lower=-1.44 upper=1.44 effort=33.5 velocity=21 -> lower=-1.5708 upper=3.4907 effort=23.7 velocity=30.1
- joint base_imu_joint: parent body -> trunk
- joint base_to_body: child body -> trunk
- joint camera_joint_front: origin xyz=0.15 0 0.05 rpy=0 0 0 -> xyz=0 0 0 rpy=0 0 0; parent body -> trunk
- joint lidar_joint: origin xyz=0 0 0.1 rpy=0 0 0 -> xyz=0 0 0 rpy=0 0 0; parent body -> trunk
