Commit message: 所有宇树接口都改成ros2话题接口，原先宇树仿真输出信息也桥接到ros2话题接口

File: src/descriptions/unitree/mybot_description/xacro/mybot/robot_body.xacro (robot description, xacro)
@@ -9,19 +9,21 @@
             <origin xyz="0 0 0" rpy="0 0 0"/>
             <parent link="base"/>
-            <child link="body"/>
-        </joint>
-        <link name="body">
+            <child link="trunk"/>
+        </joint>
+        <link name="trunk">
             <inertial>
                   <origin
-        xyz="-0.075044 0.0013153 0.023062"
+        xyz="0.0 0.0 0.0"
         rpy="0 0 0" />
                 <mass value="5.3036" />
                <inertia
-        ixx="0.012634"
-        ixy="-1.0247E-06"
-        ixz="0.002562"
-        iyy="0.017259"
-        iyz="-3.3196E-07"
-        izz="0.017164" />
+                    ixx="0.012634"
+                    ixy="-1.0247E-06"
+                    ixz="0.002562"
+                    iyy="0.017259"
+                    iyz="-3.3196E-07"
+                    izz="0.017164" />
+                <!-- go2 对应参数: trunk_mass=6.921, trunk_com=(0.021112, 0, -0.005366),
+                     inertia: ixx=0.02448, ixy=0.00012166, ixz=0.0014849, iyy=0.098077, iyz=-3.12e-05, izz=0.107 -->
             </inertial>
             <visual>
@@ -35,7 +37,8 @@
             </visual>
             <collision>
-                <origin xyz="0 0 0" rpy="0 0 0" />
-                <geometry>
-                    <mesh filename="${mesh_path}/body.STL" />
+                <!-- go2: trunk collision box size="0.3762 0.0935 0.114" -->
+                <origin xyz="0 0 0" rpy="0 0 0" />
+                <geometry>
+                    <box size="0.3762 0.0935 0.114" />
                 </geometry>
             </collision>
@@ -46,4 +49,6 @@
                 <mass value="0.62455" />
                 <inertia ixx="0.00051175" ixy="3.0689E-08" ixz="3.6249E-07" iyy="0.00080416" iyz="2.5347E-08" izz="0.00043104" />
+                <!-- go2 对应参数: hip_mass=0.678, hip_com=(-0.0054, 0.00194, -0.000105),
+                     inertia: ixx=0.00048, ixy=-3.01e-06, ixz=1.11e-06, iyy=0.000884, iyz=-1.42e-06, izz=0.000596 -->
             </inertial>
             <visual>
@@ -57,7 +62,8 @@
             </visual>
             <collision>
-                <origin xyz="0 0 0" rpy="0 0 0" />
-                <geometry>
-                    <mesh filename="${mesh_path}/FL_hip.STL" />
+                <!-- go2: hip collision cylinder radius=0.046 length=0.04 at y=+0.0955, rpy=pi/2 0 0 -->
+                <origin xyz="0 0.0955 0" rpy="1.5708 0 0" />
+                <geometry>
+                    <cylinder radius="0.046" length="0.04" />
                 </geometry>
             </collision>
@@ -65,9 +71,9 @@
         <joint name="FL_hip_joint" type="revolute">
             <origin xyz="0.0946 0.062 -0.071" rpy="0 0 0" />
-            <parent link="body" />
+            <parent link="trunk" />
             <child link="FL_hip" />
             <axis xyz="1 0 0" />
-            <!-- HAA: 侧摆关节，保持原范围 -->
-            <limit lower="-0.48" upper="0.48" effort="33.5" velocity="21" />
+            <dynamics damping="0.1" friction="0.2"/>
+            <limit lower="-1.0472" upper="1.0472" effort="23.7" velocity="30.1" />
         </joint>
         <link name="FL_thigh">
@@ -76,4 +82,6 @@
                 <mass value="1.107" />
                 <inertia ixx="0.0026249" ixy="-3.0685E-08" ixz="-3.4311E-05" iyy="0.0030336" iyz="-2.5044E-08" izz="0.00046586" />
+                <!-- go2 对应参数: thigh_mass=1.152, thigh_com=(-0.00374, -0.0223, -0.0327),
+                     inertia: ixx=0.00584, ixy=8.72e-05, ixz=-0.000289, iyy=0.0058, iyz=0.000808, izz=0.00103 -->
             </inertial>
             <visual>
@@ -87,7 +95,8 @@
             </visual>
             <collision>
-                <origin xyz="0 0 0" rpy="0 0 0" />
-                <geometry>
-                    <mesh filename="${mesh_path}/FL_thigh.STL" />
+                <!-- go2: thigh collision box size="0.213 0.0245 0.034" at z=-0.1065, rpy=0 pi/2 0 -->
+                <origin xyz="0 0 -0.1065" rpy="0 1.5708 0" />
+                <geometry>
+                    <box size="0.213 0.0245 0.034" />
                 </geometry>
             </collision>
@@ -98,6 +107,6 @@
             <child link="FL_thigh" />
             <axis xyz="0 1 0" />
-            <!-- HFE: 大腿前后摆，保持原范围 -->
-            <limit lower="-1.44" upper="1.44" effort="33.5" velocity="21" />
+            <dynamics damping="0.1" friction="0.2"/>
+            <limit lower="-1.5708" upper="3.4907" effort="23.7" velocity="30.1" />
         </joint>
         <link name="FL_calf">
@@ -106,4 +115,6 @@
                 <mass value="0.292483071997453" />
                 <inertia ixx="0.000903299669438753" ixy="-2.55525312562112E-11" ixz="0.000155678759259663" iyy="0.000949320326267258" iyz="1.05414825036111E-10" izz="6.30610325260309E-05" />
+                <!-- go2 对应参数: calf_mass=0.154, calf_com=(0.00548, -0.000975, -0.115),
+                     inertia: ixx=0.00108, ixy=3.4e-07, ixz=1.72e-05, iyy=0.0011, iyz=8.28e-06, izz=3.29e-05 -->
             </inertial>
             <visual>
@@ -117,7 +128,8 @@
             </visual>
             <collision>
-                <origin xyz="0 0 0" rpy="0 0 0" />
-                <geometry>
-                    <mesh filename="${mesh_path}/FL_calf.STL" />
+                <!-- go2: calf collision box size="0.213 0.016 0.016" at z=-0.1065, rpy=0 pi/2 0 -->
+                <origin xyz="0 0 -0.1065" rpy="0 1.5708 0" />
+                <geometry>
+                    <box size="0.213 0.016 0.016" />
                 </geometry>
             </collision>
@@ -128,6 +140,6 @@
             <child link="FL_calf" />
             <axis xyz="0 1 0" />
-            <!-- KFE: 膝关节，修改为负值区间防止反向弯折穿模 -->
-            <limit lower="-2.7" upper="-0.6" effort="33.5" velocity="21" />
+            <dynamics damping="0.1" friction="0.2"/>
+            <limit lower="-2.7227" upper="-0.83776" effort="35.55" velocity="20.06" />
         </joint>
         <link name="FL_foot">
@@ -136,4 +148,5 @@
                 <mass value="0.0335103216382911" />
                 <inertia ixx="5.36165146212658E-06" ixy="-7.94093388050967E-23" ixz="-3.17637355220363E-22" iyy="5.36165146212658E-06" iyz="1.32348898008481E-22" izz="5.36165146212658E-06" />
+                <!-- go2 对应参数: foot_mass=0.06, inertia approx ixx=iyy=izz=9.6e-06 -->
             </inertial>
             <visual>
@@ -147,12 +160,13 @@
             </visual>
             <collision>
-                <origin xyz="0 0 0" rpy="0 0 0" />
-                <geometry>
-                    <mesh filename="${mesh_path}/FL_foot.STL" />
+                <!-- go2: foot collision sphere radius=0.02 -->
+                <origin xyz="0 0 0" rpy="0 0 0" />
+                <geometry>
+                    <sphere radius="0.02" />
                 </geometry>
             </collision>
         </link>
         <joint name="FL_foot_fixed" type="fixed">
-            <origin xyz="0.0015191 -0.00024999 -0.22467" rpy="0 0 0" />
+            <origin xyz="0.0015191 -0.00025 -0.22467" rpy="0 0 0" />
             <parent link="FL_calf" />
             <child link="FL_foot" />
@@ -161,7 +175,8 @@
         <link name="FR_hip">
             <inertial>
-                <origin xyz="0.0503237105506868 -0.0023835007191014 -1.92627612935203E-05" rpy="0 0 0" />
-                <mass value="0.645332324862741" />
-                <inertia ixx="0.000516279867983271" ixy="3.06884611939023E-08" ixz="-3.62557969784867E-07" iyy="0.000812995967320655" iyz="-2.52696161538675E-08" izz="0.000435566921761248" />
+                <origin xyz="0.049109 -0.0014996 -1.9828E-05" rpy="0 0 0" />
+                <mass value="0.62455" />
+                <inertia ixx="0.00051175" ixy="3.0689E-08" ixz="3.6249E-07" iyy="0.00080416" iyz="2.5347E-08" izz="0.00043104" />
+                <!-- go2 对应参数同左前髋(镜像): hip_mass=0.678, etc. -->
             </inertial>
             <visual>
@@ -175,7 +190,8 @@
             </visual>
             <collision>
-                <origin xyz="0 0 0" rpy="0 0 0" />
-                <geometry>
-                    <mesh filename="${mesh_path}/FR_hip.STL" />
+                <!-- go2: hip collision cylinder at y=-0.0955, rpy=pi/2 0 0 -->
+                <origin xyz="0 -0.0955 0" rpy="1.5708 0 0" />
+                <geometry>
+                    <cylinder radius="0.046" length="0.04" />
                 </geometry>
             </collision>
@@ -183,14 +199,15 @@
         <joint name="FR_hip_joint" type="revolute">
             <origin xyz="0.0946 -0.062 -0.071" rpy="0 0 0" />
-            <parent link="body" />
+            <parent link="trunk" />
             <child link="FR_hip" />
             <axis xyz="1 0 0" />
-            <limit lower="-0.48" upper="0.48" effort="33.5" velocity="21" />
+            <dynamics damping="0.1" friction="0.2"/>
+            <limit lower="-1.0472" upper="1.0472" effort="23.7" velocity="30.1" />
         </joint>
         <link name="FR_thigh">
             <inertial>
-                <origin xyz="0.000368722927323942 -0.0509397168811238 -0.0448485013445288" rpy="0 0 0" />
-                <mass value="1.10704185501149" />
-                <inertia ixx="0.00262493871504934" ixy="-3.06851438667059E-08" ixz="-3.50391888175107E-05" iyy="0.00303362951335752" iyz="2.55730470397223E-08" izz="0.000465861672831916" />
+                <origin xyz="0.00040284 -0.05094 -0.044849" rpy="0 0 0" />
+                <mass value="1.107" />
+                <inertia ixx="0.0026249" ixy="-3.0685E-08" ixz="-3.4311E-05" iyy="0.0030336" iyz="-2.5044E-08" izz="0.00046586" />
             </inertial>
             <visual>
@@ -204,7 +221,7 @@
             </visual>
             <collision>
-                <origin xyz="0 0 0" rpy="0 0 0" />
-                <geometry>
-                    <mesh filename="${mesh_path}/FR_thigh.STL" />
+                <origin xyz="0 0 -0.1065" rpy="0 1.5708 0" />
+                <geometry>
+                    <box size="0.213 0.0245 0.034" />
                 </geometry>
             </collision>
@@ -215,5 +232,6 @@
             <child link="FR_thigh" />
             <axis xyz="0 1 0" />
-            <limit lower="-1.44" upper="1.44" effort="33.5" velocity="21" />
+            <dynamics damping="0.1" friction="0.2"/>
+            <limit lower="-1.5708" upper="3.4907" effort="23.7" velocity="30.1" />
         </joint>
         <link name="FR_calf">
@@ -233,7 +251,7 @@
             </visual>
             <collision>
-                <origin xyz="0 0 0" rpy="0 0 0" />
-                <geometry>
-                    <mesh filename="${mesh_path}/FR_calf.STL" />
+                <origin xyz="0 0 -0.1065" rpy="0 1.5708 0" />
+                <geometry>
+                    <box size="0.213 0.016 0.016" />
                 </geometry>
             </collision>
@@ -244,12 +262,13 @@
             <child link="FR_calf" />
             <axis xyz="0 1 0" />
-            <!-- KFE: 膝关节，修改为负值区间 -->
-            <limit lower="-2.7" upper="-0.6" effort="33.5" velocity="21" />
+            <dynamics damping="0.1" friction="0.2"/>
+            <limit lower="-2.7227" upper="-0.83776" effort="35.55" velocity="20.06" />
         </joint>
         <link name="FR_foot">
             <inertial>
-                <origin xyz="1.11022302462516E-16 -2.77555756156289E-16 2.33146835171283E-15" rpy="0 0 0" />
+                <origin xyz="0 0 0" rpy="0 0 0" />
                 <mass value="0.0335103216382911" />
                 <inertia ixx="5.36165146212658E-06" ixy="-2.68773268713706E-23" ixz="-2.7811675003655E-22" iyy="5.36165146212658E-06" iyz="2.423491454722E-23" izz="5.36165146212658E-06" />
+                <!-- go2 对应参数: foot_mass=0.06, inertia approx ixx=iyy=izz=9.6e-06 -->
             </inertial>
             <visual>
@@ -265,10 +284,10 @@
                 <origin xyz="0 0 0" rpy="0 0 0" />
                 <geometry>
-                    <mesh filename="${mesh_path}/FR_foot.STL" />
+                    <sphere radius="0.02" />
                 </geometry>
             </collision>
         </link>
         <joint name="FR_foot_fixed" type="fixed">
-            <origin xyz="0.0015191 0.00025002 -0.22467" rpy="0 0 0" />
+            <origin xyz="0.0015191 0.00025 -0.22467" rpy="0 0 0" />
             <parent link="FR_calf" />
             <child link="FR_foot" />
@@ -277,7 +296,8 @@
         <link name="RL_hip">
             <inertial>
-                <origin xyz="-0.0509369545389707 0.00155116609107588 2.07286073817398E-05" rpy="0 0 0" />
-                <mass value="0.603770938189494" />
-                <inertia ixx="0.000502920983948406" ixy="-3.06886161732306E-08" ixz="3.62490051608935E-07" iyy="0.000799637078472992" iyz="-2.52698314238679E-08" izz="0.000426513217482837" />
+                <origin xyz="-0.049109 0.0014996 1.9828E-05" rpy="0 0 0" />
+                <mass value="0.62455" />
+                <inertia ixx="0.00051175" ixy="3.0689E-08" ixz="3.6249E-07" iyy="0.00080416" iyz="2.5347E-08" izz="0.00043104" />
+                <!-- go2 对应参数(后腿镜像): hip_mass=0.678, etc. -->
             </inertial>
             <visual>
@@ -291,22 +311,24 @@
             </visual>
             <collision>
-                <origin xyz="0 0 0" rpy="0 0 0" />
-                <geometry>
-                    <mesh filename="${mesh_path}/RL_hip.STL" />
+                <!-- go2: rear-left hip collision cylinder at y=+0.0955 -->
+                <origin xyz="0 0.0955 0" rpy="1.5708 0 0" />
+                <geometry>
+                    <cylinder radius="0.046" length="0.04" />
                 </geometry>
             </collision>
         </link>
         <joint name="RL_hip_joint" type="revolute">
-            <origin xyz="-0.2146 0.062 -0.071" rpy="0 0 0" />
-            <parent link="body" />
+            <origin xyz="-0.0946 0.062 -0.071" rpy="0 0 0" />
+            <parent link="trunk" />
             <child link="RL_hip" />
             <axis xyz="1 0 0" />
-            <limit lower="-0.48" upper="0.48" effort="33.5" velocity="21" />
+            <dynamics damping="0.1" friction="0.2"/>
+            <limit lower="-1.0472" upper="1.0472" effort="23.7" velocity="30.1" />
         </joint>
         <link name="RL_thigh">
             <inertial>
-                <origin xyz="4.70856003376152E-05 0.0509397257670039 -0.0448500279170919" rpy="0 0 0" />
-                <mass value="1.10704185443719" />
-                <inertia ixx="0.00262542452560882" ixy="-3.06866137520078E-08" ixz="-2.06246560059927E-05" iyy="0.00303362951322963" iyz="-2.50435146848249E-08" izz="0.000465375862108502" />
+                <origin xyz="0.00040284 0.05094 -0.044849" rpy="0 0 0" />
+                <mass value="1.107" />
+                <inertia ixx="0.0026249" ixy="-3.0685E-08" ixz="-3.4311E-05" iyy="0.0030336" iyz="-2.5044E-08" izz="0.00046586" />
             </inertial>
             <visual>
@@ -320,7 +342,7 @@
             </visual>
             <collision>
-                <origin xyz="0 0 0" rpy="0 0 0" />
-                <geometry>
-                    <mesh filename="${mesh_path}/RL_thigh.STL" />
+                <origin xyz="0 0 -0.1065" rpy="0 1.5708 0" />
+                <geometry>
+                    <box size="0.213 0.0245 0.034" />
                 </geometry>
             </collision>
@@ -331,5 +353,6 @@
             <child link="RL_thigh" />
             <axis xyz="0 1 0" />
-            <limit lower="-1.48" upper="1.48" effort="33.5" velocity="21" />
+            <dynamics damping="0.1" friction="0.2"/>
+            <limit lower="-1.5708" upper="3.4907" effort="23.7" velocity="30.1" />
         </joint>
         <link name="RL_calf">
@@ -337,5 +360,5 @@
                 <origin xyz="0.0173313220834085 -3.8626261668756E-05 -0.100135269530252" rpy="0 0 0" />
                 <mass value="0.292483071997453" />
-                <inertia ixx="0.00090329966943877" ixy="-2.55525362041557E-11" ixz="0.000155678759259629" iyy="0.000949320326267271" iyz="1.05414855252192E-10" izz="6.30610325260272E-05" />
+                <inertia ixx="0.000903299669438753" ixy="-2.55525312562112E-11" ixz="0.000155678759259663" iyy="0.000949320326267258" iyz="1.05414825036111E-10" izz="6.30610325260309E-05" />
             </inertial>
             <visual>
@@ -349,7 +372,7 @@
             </visual>
             <collision>
-                <origin xyz="0 0 0" rpy="0 0 0" />
-                <geometry>
-                    <mesh filename="${mesh_path}/RL_calf.STL" />
+                <origin xyz="0 0 -0.1065" rpy="0 1.5708 0" />
+                <geometry>
+                    <box size="0.213 0.016 0.016" />
                 </geometry>
             </collision>
@@ -360,12 +383,13 @@
             <child link="RL_calf" />
             <axis xyz="0 1 0" />
-            <!-- KFE: 膝关节，修改为负值区间 -->
-            <limit lower="-2.7" upper="-0.6" effort="33.5" velocity="21" />
+            <dynamics damping="0.1" friction="0.2"/>
+            <limit lower="-2.7227" upper="-0.83776" effort="35.55" velocity="20.06" />
         </joint>
         <link name="RL_foot">
             <inertial>
-                <origin xyz="7.43849426498855E-15 2.22044604925031E-16 -7.88258347483861E-15" rpy="0 0 0" />
+                <origin xyz="0 0 0" rpy="0 0 0" />
                 <mass value="0.0335103216382911" />
-                <inertia ixx="5.36165146212658E-06" ixy="4.2351647362715E-22" ixz="5.29395592033912E-23" iyy="5.36165146212658E-06" iyz="1.58818677610181E-22" izz="5.36165146212658E-06" />
+                <inertia ixx="5.36165146212658E-06" ixy="-7.94093388050967E-23" ixz="-3.17637355220363E-22" iyy="5.36165146212658E-06" iyz="1.32348898008481E-22" izz="5.36165146212658E-06" />
+                <!-- go2 对应参数: foot_mass=0.06, inertia approx ixx=iyy=izz=9.6e-06 -->
             </inertial>
             <visual>
@@ -381,10 +405,10 @@
                 <origin xyz="0 0 0" rpy="0 0 0" />
                 <geometry>
-                    <mesh filename="${mesh_path}/RL_foot.STL" />
+                    <sphere radius="0.02" />
                 </geometry>
             </collision>
         </link>
         <joint name="RL_foot_fixed" type="fixed">
-            <origin xyz="0.0015191 -0.00024998 -0.22467" rpy="0 0 0" />
+            <origin xyz="0.0015191 -0.00025 -0.22467" rpy="0 0 0" />
             <parent link="RL_calf" />
             <child link="RL_foot" />
@@ -393,7 +417,8 @@
         <link name="RR_hip">
             <inertial>
-                <origin xyz="0 0 0" rpy="0 0 0" />
-                <mass value="0" />
-                <inertia ixx="0" ixy="0" ixz="0" iyy="0" iyz="0" izz="0" />
+                <origin xyz="-0.049109 -0.0014996 1.9828E-05" rpy="0 0 0" />
+                <mass value="0.62455" />
+                <inertia ixx="0.00051175" ixy="3.0689E-08" ixz="3.6249E-07" iyy="0.00080416" iyz="2.5347E-08" izz="0.00043104" />
+                <!-- go2 对应参数(后腿镜像): hip_mass=0.678, etc. -->
             </inertial>
             <visual>
@@ -407,22 +432,24 @@
             </visual>
             <collision>
-                <origin xyz="0 0 0" rpy="0 0 0" />
-                <geometry>
-                    <mesh filename="${mesh_path}/RR_hip.STL" />
+                <!-- go2: rear-right hip collision cylinder at y=-0.0955 -->
+                <origin xyz="0 -0.0955 0" rpy="1.5708 0 0" />
+                <geometry>
+                    <cylinder radius="0.046" length="0.04" />
                 </geometry>
             </collision>
         </link>
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
File: src/descriptions/unitree/mybot_description/xacro/robot.xacro (robot description, xacro)
@@ -23,6 +23,6 @@
     <xacro:include filename="$(find mybot_description)/xacro/ros2_control.xacro"/>
   </xacro:unless>
-  <!-- 网格文件路径 -->
-  <xacro:property name="mesh_path" value="$(find mybot_description)/meshes"/>
+  <!-- 网格文件路径（使用 package:// 以兼容资源检索） -->
+  <xacro:property name="mesh_path" value="package://mybot_description/meshes"/>
   <!-- Debug 模式：固定机器人到世界坐标系 -->
   <xacro:if value="$(arg DEBUG)">
@@ -37,11 +37,11 @@
   <xacro:mybot_body mesh_path="${mesh_path}"/>
   <!-- IMU 传感器 -->
-  <xacro:IMU connected_to="body" imu_name="base_imu" xyz="0 0 0" rpy="0 0 0"/>
+  <xacro:IMU connected_to="trunk" imu_name="base_imu" xyz="0 0 0" rpy="0 0 0"/>
   <!-- 前置相机 (可选) -->
   <xacro:if value="$(arg USE_CAMERA)">
     <joint name="camera_joint_front" type="fixed">
-      <parent link="body"/>
+      <parent link="trunk"/>
       <child link="front_camera"/>
-      <origin rpy="0 0 0" xyz="0.15 0 0.05"/>
+      <origin rpy="0 0 0" xyz="0 0 0"/>
     </joint>
     <link name="front_camera">
@@ -63,7 +63,7 @@
   <xacro:if value="$(arg USE_LIDAR)">
     <joint name="lidar_joint" type="fixed">
-      <parent link="body"/>
+      <parent link="trunk"/>
       <child link="lidar"/>
-      <origin rpy="0 0 0" xyz="0 0 0.1"/>
+      <origin rpy="0 0 0" xyz="0 0 0"/>
     </joint>
     <link name="lidar">

File: src/descriptions/unitree/mybot_description/xacro/ros2_control.xacro (robot description, xacro)
@@ -4,7 +4,12 @@
 		<hardware>
 			<plugin>hardware_unitree_mujoco/HardwareUnitree</plugin>
-<!--			<param name="domain">0</param>-->
-<!--			<param name="network_interface">enp46s0</param>-->
-<!--			<param name="show_foot_force">true</param>-->
+			<!-- All IO via ROS topics (DDS-free) -->
+			<param name="state_joint_topic">/joint_states</param>
+			<param name="state_imu_topic">/imu</param>
+			<param name="state_foot_force_topic">/foot_force</param>
+			<param name="state_odometry_topic">/odometry</param>
+			<param name="command_joint_topic">/joint_command</param>
+			<param name="command_kp_topic">/joint_kp</param>
+			<param name="command_kd_topic">/joint_kd</param>
 		</hardware>
 		<joint name="FR_hip_joint">
@@ -141,8 +146,9 @@
 		</sensor>
 		<sensor name="foot_force">
+			<!-- Order aligned to controller config: FL, RL, FR, RR -->
+			<state_interface name="FL"/>
+			<state_interface name="RL"/>
 			<state_interface name="FR"/>
-			<state_interface name="FL"/>
 			<state_interface name="RR"/>
-			<state_interface name="RL"/>
 		</sensor>
 		<sensor name="odometer">
