Commit message: 添加了一些调试代码 上实际机器人测试效果目前很一般

File: src/descriptions/unitree/go2_description/xacro/ros2_control.xacro (robot description, xacro)
@@ -6,5 +6,7 @@
 			<!-- All IO via ROS topics (DDS-free) -->
 			<param name="state_joint_topic">/joint_states</param>
-			<param name="state_imu_topic">/imu</param>
+			<param name="state_imu_topic">/livox/imu</param>
+			<!-- IMU acceleration is provided in g; convert to m/s^2 in hardware -->
+			<param name="imu_linear_accel_in_g">true</param>
 			<param name="state_foot_force_topic">/foot_force</param>
 			<param name="state_odometry_topic">/odometry</param>
@@ -73,4 +75,34 @@
 			<state_interface name="effort"/>
 		</joint>
+		<joint name="RL_hip_joint">
+			<command_interface name="position"/>
+			<command_interface name="velocity"/>
+			<command_interface name="effort"/>
+			<command_interface name="kp"/>
+			<command_interface name="kd"/>
+			<state_interface name="position"/>
+			<state_interface name="velocity"/>
+			<state_interface name="effort"/>
+		</joint>
+		<joint name="RL_thigh_joint">
+			<command_interface name="position"/>
+			<command_interface name="velocity"/>
+			<command_interface name="effort"/>
+			<command_interface name="kp"/>
+			<command_interface name="kd"/>
+			<state_interface name="position"/>
+			<state_interface name="velocity"/>
+			<state_interface name="effort"/>
+		</joint>
+		<joint name="RL_calf_joint">
+			<command_interface name="position"/>
+			<command_interface name="velocity"/>
+			<command_interface name="effort"/>
+			<command_interface name="kp"/>
+			<command_interface name="kd"/>
+			<state_interface name="position"/>
+			<state_interface name="velocity"/>
+			<state_interface name="effort"/>
+		</joint>
 		<joint name="RR_hip_joint">
 			<command_interface name="position"/>
@@ -94,34 +126,4 @@
 		</joint>
 		<joint name="RR_calf_joint">
-			<command_interface name="position"/>
-			<command_interface name="velocity"/>
-			<command_interface name="effort"/>
-			<command_interface name="kp"/>
-			<command_interface name="kd"/>
-			<state_interface name="position"/>
-			<state_interface name="velocity"/>
-			<state_interface name="effort"/>
-		</joint>
-		<joint name="RL_hip_joint">
-			<command_interface name="position"/>
-			<command_interface name="velocity"/>
-			<command_interface name="effort"/>
-			<command_interface name="kp"/>
-			<command_interface name="kd"/>
-			<state_interface name="position"/>
-			<state_interface name="velocity"/>
-			<state_interface name="effort"/>
-		</joint>
-		<joint name="RL_thigh_joint">
-			<command_interface name="position"/>
-			<command_interface name="velocity"/>
-			<command_interface name="effort"/>
-			<command_interface name="kp"/>
-			<command_interface name="kd"/>
-			<state_interface name="position"/>
-			<state_interface name="velocity"/>
-			<state_interface name="effort"/>
-		</joint>
-		<joint name="RL_calf_joint">
 			<command_interface name="position"/>
 			<command_interface name="velocity"/>

File: src/descriptions/unitree/mybot_description/xacro/ros2_control.xacro (robot description, xacro)
@@ -73,4 +73,34 @@
 			<state_interface name="effort"/>
 		</joint>
+		<joint name="RL_hip_joint">
+			<command_interface name="position"/>
+			<command_interface name="velocity"/>
+			<command_interface name="effort"/>
+			<command_interface name="kp"/>
+			<command_interface name="kd"/>
+			<state_interface name="position"/>
+			<state_interface name="velocity"/>
+			<state_interface name="effort"/>
+		</joint>
+		<joint name="RL_thigh_joint">
+			<command_interface name="position"/>
+			<command_interface name="velocity"/>
+			<command_interface name="effort"/>
+			<command_interface name="kp"/>
+			<command_interface name="kd"/>
+			<state_interface name="position"/>
+			<state_interface name="velocity"/>
+			<state_interface name="effort"/>
+		</joint>
+		<joint name="RL_calf_joint">
+			<command_interface name="position"/>
+			<command_interface name="velocity"/>
+			<command_interface name="effort"/>
+			<command_interface name="kp"/>
+			<command_interface name="kd"/>
+			<state_interface name="position"/>
+			<state_interface name="velocity"/>
+			<state_interface name="effort"/>
+		</joint>
 		<joint name="RR_hip_joint">
 			<command_interface name="position"/>
@@ -94,34 +124,4 @@
 		</joint>
 		<joint name="RR_calf_joint">
-			<command_interface name="position"/>
-			<command_interface name="velocity"/>
-			<command_interface name="effort"/>
-			<command_interface name="kp"/>
-			<command_interface name="kd"/>
-			<state_interface name="position"/>
-			<state_interface name="velocity"/>
-			<state_interface name="effort"/>
-		</joint>
-		<joint name="RL_hip_joint">
-			<command_interface name="position"/>
-			<command_interface name="velocity"/>
-			<command_interface name="effort"/>
-			<command_interface name="kp"/>
-			<command_interface name="kd"/>
-			<state_interface name="position"/>
-			<state_interface name="velocity"/>
-			<state_interface name="effort"/>
-		</joint>
-		<joint name="RL_thigh_joint">
-			<command_interface name="position"/>
-			<command_interface name="velocity"/>
-			<command_interface name="effort"/>
-			<command_interface name="kp"/>
-			<command_interface name="kd"/>
-			<state_interface name="position"/>
-			<state_interface name="velocity"/>
-			<state_interface name="effort"/>
-		</joint>
-		<joint name="RL_calf_joint">
 			<command_interface name="position"/>
 			<command_interface name="velocity"/>

Commit message: 修改切换步态的时候的足端判断，防止初始化的默认swingall导致坏帧。

File: src/descriptions/unitree/go2_description/xacro/ros2_control.xacro (robot description, xacro)
@@ -4,14 +4,7 @@
 		<hardware>
 			<plugin>hardware_unitree_mujoco/HardwareUnitree</plugin>
-			<!-- All IO via ROS topics (DDS-free) -->
-			<param name="state_joint_topic">/joint_states</param>
-			<param name="state_imu_topic">/livox/imu</param>
-			<!-- IMU acceleration is provided in g; convert to m/s^2 in hardware -->
-			<param name="imu_linear_accel_in_g">true</param>
-			<param name="state_foot_force_topic">/foot_force</param>
-			<param name="state_odometry_topic">/odometry</param>
-			<param name="command_joint_topic">/joint_command</param>
-			<param name="command_kp_topic">/joint_kp</param>
-			<param name="command_kd_topic">/joint_kd</param>
+<!--			<param name="domain">0</param>-->
+<!--			<param name="network_interface">enp46s0</param>-->
+<!--			<param name="show_foot_force">true</param>-->
 		</hardware>
 		<joint name="FR_hip_joint">

File: src/descriptions/unitree/mybot_description/urdf/robot.urdf (robot description, URDF)
Before this commit: robot mybot, 21 links, 20 joints
Links:
- link trunk: mass 5.3036 -> 4.30616163

File: src/descriptions/unitree/mybot_description/xacro/ros2_control.xacro (robot description, xacro)
@@ -9,7 +9,7 @@
 			<param name="state_foot_force_topic">/foot_force</param>
 			<param name="state_odometry_topic">/odometry</param>
-			<param name="command_joint_topic">/joint_command</param>
-			<param name="command_kp_topic">/joint_kp</param>
-			<param name="command_kd_topic">/joint_kd</param>
+			<param name="command_joint_topic">/joint_commands</param>
+			<param name="command_kp_topic">/kp_commands</param>
+			<param name="command_kd_topic">/kd_commands</param>
 		</hardware>
 		<joint name="FR_hip_joint">
