Commit message: 这个版本可以跑mujoco

File: src/descriptions/unitree/mybot_description/urdf/robot.urdf (robot description, URDF)
Before this commit: robot go2, 19 links, 18 joints
Links:
- removed link imu_link
- removed link trunk
- added link base_imu, mass 0.01; visual box size=0.015 0.015 0.004
- added link body, mass 5.3036; collision mesh filename=/home/rc_kfs/quadruped_ros2_control/install/mybot_descripti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; visual mesh filename=/home/rc_kfs/quadruped_ros2_control/install/mybot_descripti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
- added link front_camera, mass 0.1; visual box size=0.05 0.05 0.05
- added link lidar, mass 0.2; collision cylinder length=0.07 radius=0.04; visual cylinder length=0.07 radius=0.04
- link FL_calf: mass 0.154 -> 0.292483071997453; geometry collision mesh filename=/home/rc_kfs/quadruped_ros2_control/install/mybot_descripti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; visual mesh filename=/home/rc_kfs/quadruped_ros2_control/install/mybot_descripti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
- link FL_foot: mass 0.06 -> 0.0335103216382911; geometry collision mesh filename=/home/rc_kfs/quadruped_ros2_control/install/mybot_descripti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; visual mesh filename=/home/rc_kfs/quadruped_ros2_control/install/mybot_descripti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
- link FL_hip: mass 0.678 -> 0.62455; geometry collision mesh filename=/home/rc_kfs/quadruped_ros2_control/install/mybot_descripti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; visual mesh filename=/home/rc_kfs/quadruped_ros2_control/install/mybot_descripti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
- link FL_thigh: mass 1.152 -> 1.107; geometry collision mesh filename=/home/rc_kfs/quadruped_ros2_control/install/mybot_descripti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; visual mesh filename=/home/rc_kfs/quadruped_ros2_control/install/mybot_descripti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
- link FR_calf: mass 0.154 -> 0.292483071997452; geometry collision mesh filename=/home/rc_kfs/quadruped_ros2_control/install/mybot_descripti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; visual mesh filename=/home/rc_kfs/quadruped_ros2_control/install/mybot_descripti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
- link FR_foot: mass 0.06 -> 0.0335103216382911; geometry collision mesh filename=/home/rc_kfs/quadruped_ros2_control/install/mybot_descripti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; visual mesh filename=/home/rc_kfs/quadruped_ros2_control/install/mybot_descripti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
- link FR_hip: mass 0.678 -> 0.645332324862741; geometry collision mesh filename=/home/rc_kfs/quadruped_ros2_control/install/mybot_descripti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; visual mesh filename=/home/rc_kfs/quadruped_ros2_control/install/mybot_descripti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
- link FR_thigh: mass 1.152 -> 1.10704185501149; geometry collision mesh filename=/home/rc_kfs/quadruped_ros2_control/install/mybot_descripti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; visual mesh filename=/home/rc_kfs/quadruped_ros2_control/install/mybot_descripti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
- link RL_calf: mass 0.154 -> 0.292483071997453; geometry collision mesh filename=/home/rc_kfs/quadruped_ros2_control/install/mybot_descripti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; visual mesh filename=/home/rc_kfs/quadruped_ros2_control/install/mybot_descripti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
- link RL_foot: mass 0.06 -> 0.0335103216382911; geometry collision mesh filename=/home/rc_kfs/quadruped_ros2_control/install/mybot_descripti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; visual mesh filename=/home/rc_kfs/quadruped_ros2_control/install/mybot_descripti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
- link RL_hip: mass 0.678 -> 0.603770938189494; geometry collision mesh filename=/home/rc_kfs/quadruped_ros2_control/install/mybot_descripti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; visual mesh filename=/home/rc_kfs/quadruped_ros2_control/install/mybot_descripti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
- link RL_thigh: mass 1.152 -> 1.10704185443719; geometry collision mesh filename=/home/rc_kfs/quadruped_ros2_control/install/mybot_descripti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; visual mesh filename=/home/rc_kfs/quadruped_ros2_control/install/mybot_descripti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
- link RR_calf: mass 0.154 -> 0.292483071997453; geometry collision mesh filename=/home/rc_kfs/quadruped_ros2_control/install/mybot_descripti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; visual mesh filename=/home/rc_kfs/quadruped_ros2_control/install/mybot_descripti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
- link RR_foot: mass 0.06 -> 0.0335103216382911; geometry collision mesh filename=/home/rc_kfs/quadruped_ros2_control/install/mybot_descripti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; visual mesh filename=/home/rc_kfs/quadruped_ros2_control/install/mybot_descripti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
- link RR_hip: mass 0.678 -> 0; geometry collision mesh filename=/home/rc_kfs/quadruped_ros2_control/install/mybot_descripti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; visual mesh filename=/home/rc_kfs/quadruped_ros2_control/install/mybot_descripti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
- link RR_thigh: mass 1.152 -> 1.10704185429829; geometry collision mesh filename=/home/rc_kfs/quadruped_ros2_control/install/mybot_descripti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; visual mesh filename=/home/rc_kfs/quadruped_ros2_control/install/mybot_descripti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
- link base: geometry 
Joints:
- removed joint floating_base
- removed joint imu_joint
- added joint base_imu_joint: type fixed, parent body, child base_imu, origin xyz=0 0 0 rpy=0 0 0
- added joint base_to_body: type fixed, parent base, child body, origin xyz=0 0 0 rpy=0 0 0
- added joint camera_joint_front: type fixed, parent body, child front_camera, origin xyz=0.15 0 0.05 rpy=0 0 0
- added joint lidar_joint: type fixed, parent body, child lidar, origin xyz=0 0 0.1 rpy=0 0 0
- joint FL_calf_joint: limit lower=-2.7227 upper=-0.83776 effort=35.55 velocity=20.06 -> lower=-2.7 upper=-0.6 effort=33.5 velocity=21; origin xyz=0 0 -0.213 rpy=0 -0 0 -> xyz=0 0.0705 -0.22 rpy=0 0 0
- joint FL_foot_fixed: origin xyz=0 0 -0.213 rpy=0 -0 0 -> xyz=0.0015191 -0.00024999 -0.22467 rpy=0 0 0
- joint FL_hip_joint: limit lower=-1.0472 upper=1.0472 effort=23.7 velocity=30.1 -> lower=-0.48 upper=0.48 effort=33.5 velocity=21; origin xyz=0.1934 0.0465 0 rpy=0 -0 0 -> xyz=0.0946 0.062 -0.071 rpy=0 0 0; parent trunk -> body
- joint FL_thigh_joint: limit lower=-1.5708 upper=3.4907 effort=23.7 velocity=30.1 -> lower=-1.44 upper=1.44 effort=33.5 velocity=21; origin xyz=0 0.0955 0 rpy=0 -0 0 -> xyz=0.085 0.03295 0 rpy=0 0 0
- joint FR_calf_joint: limit lower=-2.7227 upper=-0.83776 effort=35.55 velocity=20.06 -> lower=-2.7 upper=-0.6 effort=33.5 velocity=21; origin xyz=0 0 -0.213 rpy=0 -0 0 -> xyz=0 -0.0705 -0.22 rpy=0 0 0
- joint FR_foot_fixed: origin xyz=0 0 -0.213 rpy=0 -0 0 -> xyz=0.0015191 0.00025002 -0.22467 rpy=0 0 0
- joint FR_hip_joint: limit lower=-1.0472 upper=1.0472 effort=23.7 velocity=30.1 -> lower=-0.48 upper=0.48 effort=33.5 velocity=21; origin xyz=0.1934 -0.0465 0 rpy=0 -0 0 -> xyz=0.0946 -0.062 -0.071 rpy=0 0 0; parent trunk -> body
- joint FR_thigh_joint: limit lower=-1.5708 upper=3.4907 effort=23.7 velocity=30.1 -> lower=-1.44 upper=1.44 effort=33.5 velocity=21; origin xyz=0 -0.0955 0 rpy=0 -0 0 -> xyz=0.085 -0.03295 0 rpy=0 0 0
- joint RL_calf_joint: limit lower=-2.7227 upper=-0.83776 effort=35.55 velocity=20.06 -> lower=-2.7 upper=-0.6 effort=33.5 velocity=21; origin xyz=0 0 -0.213 rpy=0 -0 0 -> xyz=0 0.0705 -0.22 rpy=0 0 0
- joint RL_foot_fixed: origin xyz=0 0 -0.213 rpy=0 -0 0 -> xyz=0.0015191 -0.00024998 -0.22467 rpy=0 0 0
- joint RL_hip_joint: limit lower=-1.0472 upper=1.0472 effort=23.7 velocity=30.1 -> lower=-0.48 upper=0.48 effort=33.5 velocity=21; origin xyz=-0.1934 0.0465 0 rpy=0 -0 0 -> xyz=-0.2146 0.062 -0.071 rpy=0 0 0; parent trunk -> body
- joint RL_thigh_joint: limit lower=-1.5708 upper=3.4907 effort=23.7 velocity=30.1 -> lower=-1.48 upper=1.48 effort=33.5 velocity=21; origin xyz=0 0.0955 0 rpy=0 -0 0 -> xyz=-0.085 0.03295 0 rpy=0 0 0
- joint RR_calf_joint: limit lower=-2.7227 upper=-0.83776 effort=35.55 velocity=20.06 -> lower=-2.7 upper=-0.6 effort=33.5 velocity=21; origin xyz=0 0 -0.213 rpy=0 -0 0 -> xyz=0 -0.0705 -0.22 rpy=0 0 0
- joint RR_foot_fixed: origin xyz=0 0 -0.213 rpy=0 -0 0 -> xyz=0.0015191 0.00025002 -0.22467 rpy=0 0 0
- joint RR_hip_joint: limit lower=-1.0472 upper=1.0472 effort=23.7 velocity=30.1 -> lower=-0.48 upper=0.48 effort=33.5 velocity=21; origin xyz=-0.1934 -0.0465 0 rpy=0 -0 0 -> xyz=-0.2146 -0.062 -0.071 rpy=0 0 0; parent trunk -> body
- joint RR_thigh_joint: limit lower=-1.5708 upper=3.4907 effort=23.7 velocity=30.1 -> lower=-1.44 upper=1.44 effort=33.5 velocity=21; origin xyz=0 -0.0955 0 rpy=0 -0 0 -> xyz=-0.085 -0.03295 0 rpy=0 0 0

File: src/descriptions/unitree/mybot_description/xacro/robot.xacro (robot description, xacro)
@@ -1,10 +1,15 @@
 <?xml version="1.0"?>
 <robot name="mybot" xmlns:xacro="http://www.ros.org/wiki/xacro">
+  <!-- 配置参数 -->
   <xacro:arg name="DEBUG" default="false"/>
   <xacro:arg name="GAZEBO" default="false"/>
   <xacro:arg name="CLASSIC" default="false"/>
-  <xacro:include filename="$(find mybot_description)/xacro/const.xacro"/>
-  <xacro:include filename="$(find mybot_description)/xacro/materials.xacro"/>
-  <xacro:include filename="$(find mybot_description)/xacro/leg.xacro"/>
+  <xacro:arg name="USE_CAMERA" default="true"/>
+  <xacro:arg name="USE_LIDAR" default="true"/>
+  <!-- 包含 mybot 配置文件 -->
+  <xacro:include filename="$(find mybot_description)/xacro/my_common/materials.xacro"/>
+  <xacro:include filename="$(find mybot_description)/xacro/my_common/imu.xacro"/>
+  <xacro:include filename="$(find mybot_description)/xacro/mybot/robot_body.xacro"/>
+  <!-- Gazebo 或控制器配置 -->
   <xacro:if value="$(arg GAZEBO)">
     <xacro:if value="$(arg CLASSIC)">
@@ -18,8 +23,7 @@
     <xacro:include filename="$(find mybot_description)/xacro/ros2_control.xacro"/>
   </xacro:unless>
-  <!-- <xacro:stairs stairs="15" xpos="0" ypos="0" zpos="0" /> -->
-  <!-- Rotor related joint and link is only for demonstrate location. -->
-  <!-- Actually, the rotor will rotate and the joint is not fixed. Reduction ratio should be considered. -->
-  <!-- Debug mode will hung up the robot, use "true" or "false" to switch it. -->
+  <!-- 网格文件路径 -->
+  <xacro:property name="mesh_path" value="$(find mybot_description)/meshes"/>
+  <!-- Debug 模式：固定机器人到世界坐标系 -->
   <xacro:if value="$(arg DEBUG)">
     <link name="world"/>
@@ -30,102 +34,57 @@
     </joint>
   </xacro:if>
-  <link name="base">
-    <visual>
-      <origin rpy="0 0 0" xyz="0 0 0"/>
-      <geometry>
-        <box size="0.001 0.001 0.001"/>
-      </geometry>
-    </visual>
-  </link>
-  <joint name="floating_base" type="fixed">
-    <origin rpy="0 0 0" xyz="0 0 0"/>
-    <parent link="base"/>
-    <child link="trunk"/>
-  </joint>
-  <link name="trunk">
-    <visual>
-      <origin rpy="0 0 0" xyz="0 0 0"/>
-      <geometry>
-        <mesh filename="file://$(find mybot_description)/meshes/trunk.dae" scale="1 1 1"/>
-      </geometry>
-      <!-- <material name="orange"/> -->
-    </visual>
-    <collision>
-      <origin rpy="0 0 0" xyz="0 0 0"/>
-      <geometry>
-        <box size="${trunk_length} ${trunk_width} ${trunk_height}"/>
-      </geometry>
-    </collision>
-    <collision>
-      <origin rpy="0 0 0" xyz="0 0 0"/>
-      <geometry>
-        <box size="0.1881 0.04675 0.057"/>
-      </geometry>
-    </collision>
-    <collision>
-      <origin rpy="0 0 0" xyz="0.285 0 0.01"/>
-      <geometry>
-        <cylinder length="0.05" radius="0.045"/>
-      </geometry>
-    </collision>
-    <collision>
-      <origin rpy="0 0 0" xyz="0.293 0 -0.06"/>
-      <geometry>
-        <box size="0.047 0.047 0.047"/>
-      </geometry>
-    </collision>
-    <inertial>
-      <origin rpy="0 0 0" xyz="${trunk_com_x} ${trunk_com_y} ${trunk_com_z}"/>
-      <mass value="${trunk_mass}"/>
-      <inertia
-          ixx="${trunk_ixx}" ixy="${trunk_ixy}" ixz="${trunk_ixz}"
-          iyy="${trunk_iyy}" iyz="${trunk_iyz}"
-          izz="${trunk_izz}"/>
-    </inertial>
-  </link>
-  <joint name="imu_joint" type="fixed">
-    <parent link="trunk"/>
-    <child link="imu_link"/>
-    <origin rpy="0 0 0" xyz="0 0 0"/>
-  </joint>
-  <link name="imu_link">
-    <inertial>
-      <mass value="0.001"/>
-      <origin rpy="0 0 0" xyz="0 0 0"/>
-      <inertia ixx="0.0001" ixy="0" ixz="0" iyy="0.0001" iyz="0" izz="0.0001"/>
-    </inertial>
-    <visual>
-      <origin rpy="0 0 0" xyz="0 0 0"/>
-      <geometry>
-        <box size="0.001 0.001 0.001"/>
-      </geometry>
-      <!-- <material name="red"/> -->
-    </visual>
-    <collision>
-      <origin rpy="0 0 0" xyz="0 0 0"/>
-      <geometry>
-        <box size=".001 .001 .001"/>
-      </geometry>
-    </collision>
-  </link>
-  <joint name="camera_joint_front" type="fixed">
-    <parent link="trunk"/>
-    <child link="front_camera"/>
-    <origin rpy="0 0 0" xyz="0.32715 0 0.04297"/>
-  </joint>
-  <link name="front_camera">
-  </link>
-  <joint name="lidar_joint" type="fixed">
-    <origin
-        xyz="0.28945 0 -0.046825" rpy="0 2.8782 0"/>
-    <parent link="trunk"/>
-    <child link="lidar"/>
-    <axis xyz="0 0 0"/>
-  </joint>
-  <link name="lidar">
-  </link>
-  <xacro:leg name="FR" mirror="-1" mirror_dae="False" front_hind="1" front_hind_dae="True"/>
-  <xacro:leg name="FL" mirror="1" mirror_dae="True" front_hind="1" front_hind_dae="True"/>
-  <xacro:leg name="RR" mirror="-1" mirror_dae="False" front_hind="-1" front_hind_dae="False"/>
-  <xacro:leg name="RL" mirror="1" mirror_dae="True" front_hind="-1" front_hind_dae="False"/>
+  <!-- 创建 mybot 机器人主体和腿部 -->
+  <xacro:mybot_body mesh_path="${mesh_path}"/>
+  <!-- IMU 传感器 -->
+  <xacro:IMU connected_to="body" imu_name="base_imu" xyz="0 0 0" rpy="0 0 0"/>
+  <!-- 前置相机 (可选) -->
+  <xacro:if value="$(arg USE_CAMERA)">
+    <joint name="camera_joint_front" type="fixed">
+      <parent link="body"/>
+      <child link="front_camera"/>
+      <origin rpy="0 0 0" xyz="0.15 0 0.05"/>
+    </joint>
+    <link name="front_camera">
+      <inertial>
+        <mass value="0.1"/>
+        <origin rpy="0 0 0" xyz="0 0 0"/>
+        <inertia ixx="0.00001" ixy="0" ixz="0" iyy="0.00001" iyz="0" izz="0.00001"/>
+      </inertial>
+      <visual>
+        <origin rpy="0 0 0" xyz="0 0 0"/>
+        <geometry>
+          <box size="0.05 0.05 0.05"/>
+        </geometry>
+        <material name="grey"/>
+      </visual>
+    </link>
+  </xacro:if>
+  <!-- LIDAR 传感器 (可选) -->
+  <xacro:if value="$(arg USE_LIDAR)">
+    <joint name="lidar_joint" type="fixed">
+      <parent link="body"/>
+      <child link="lidar"/>
+      <origin rpy="0 0 0" xyz="0 0 0.1"/>
+    </joint>
+    <link name="lidar">
+      <inertial>
+        <mass value="0.2"/>
+        <origin rpy="0 0 0" xyz="0 0 0"/>
+        <inertia ixx="0.00002" ixy="0" ixz="0" iyy="0.00002" iyz="0" izz="0.00002"/>
+      </inertial>
+      <visual>
+        <origin rpy="0 0 0" xyz="0 0 0"/>
+        <geometry>
+          <cylinder radius="0.04" length="0.07"/>
+        </geometry>
+        <material name="black"/>
+      </visual>
+      <collision>
+        <origin rpy="0 0 0" xyz="0 0 0"/>
+        <geometry>
+          <cylinder radius="0.04" length="0.07"/>
+        </geometry>
+      </collision>
+    </link>
+  </xacro:if>
 </robot>
